Commit message: launch file created

File: src/myrobot2_description/urdf/myrobot2.urdf (robot description, URDF)
Before this commit: robot myrobot2, 4 links, 3 joints
Links:
- removed link base_footlink
- added link base_footprint
Joints:
- joint base_joint: origin xyz=0.0 0.0 0.0 rpy=0.0 0.0 0.055 -> xyz=0.0 0.0 0.055 rpy=0.0 0.0 0.0
